File: StepDriver.sch (KiCad schematic (older format))
At the start: 48 parts, among them IC1 MCP25625-E_ML, J1 SW, J2 Conn_01x05, J3 SERIAL, J4 ICSP, J5 I2C, J7 Terminals_01x04, J8 ENCODER, Q1 SI3415A, SW1 SW_DIP_x01, U1 ATMEGA328P-AU, U2 uA7805, Y1 OSCILLATOR-16MHZ, Y2 OSCILLATOR-16MHZ

Commit message: Small changes, added step and refined schematic and images
Parts:
- A1: symbol Pololu_Breakout_A4988 -> StepDriver-rescue:Pololu_Breakout_A4988
- C1, C10, C11, C12, C13, C14, C3, C4, C5, C6, C7, C8, C9: symbol C -> StepDriver-rescue:C
- C15, C2: symbol CP -> StepDriver-rescue:CP
- D1, D2: symbol LED -> StepDriver-rescue:LED
- IC1: symbol MCP25625-E_ML -> MCP25625-E_ML:MCP25625-E_ML
- J1, J3, J8: symbol Conn_01x04 -> StepDriver-rescue:Conn_01x04
- J2: symbol Conn_01x05 -> StepDriver-rescue:Conn_01x05
- J4: symbol Conn_02x03_Counter_Clockwise -> StepDriver-rescue:Conn_02x03_Counter_Clockwise
- J5: symbol Conn_02x02_Counter_Clockwise -> StepDriver-rescue:Conn_02x02_Counter_Clockwise
- J7: symbol Screw_Terminal_01x04 -> StepDriver-rescue:Screw_Terminal_01x04
- MK1, MK2, MK3, MK4: symbol Mounting_Hole -> StepDriver-rescue:Mounting_Hole
- Q1: symbol Q_PMOS_GSD -> StepDriver-rescue:Q_PMOS_GSD
- R1, R10, R11, R2, R3, R4, R5, R6, R7, R8, R9: symbol R -> StepDriver-rescue:R
- SW1: symbol SW_DIP_x01 -> StepDriver-rescue:SW_DIP_x01
- TP2: symbol TEST -> StepDriver-rescue:TEST
- U1: symbol ATMEGA328P-AU -> StepDriver-rescue:ATMEGA328P-AU
- U2: symbol uA7805 -> StepDriver-rescue:uA7805
- Y1, Y2: symbol OSCILLATOR-16MHZSMD-7X5-4PAD -> SparkFun-Clocks:OSCILLATOR-16MHZSMD-7X5-4PAD
Other:
- note added: "Short R11"
- note removed: "Power for the\nCAN controller"
